Commit message: feat: add dummy root

File: pnp_dual_fr3_description/robots/pnp_dual_fr3/pnp_dual_fr3.srdf.xacro (robot description, xacro)
@@ -126,5 +126,5 @@
     <joint name="${right_full_prefix}joint7" value="${home_positions.right.joint7}"/>
   </group_state>
-  <virtual_joint name="world_joint" type="fixed" parent_frame="world" child_link="base_link"/>
+  <virtual_joint name="world_joint" type="fixed" parent_frame="world" child_link="pnp_root"/>
   <xacro:standard_arm_collisions full_arm_prefix="${left_full_prefix}"/>
   <xacro:extra_arm_collisions full_arm_prefix="${left_full_prefix}"/>

File: pnp_dual_fr3_description/robots/pnp_dual_fr3/pnp_dual_fr3.urdf.xacro (robot description, xacro)
@@ -34,4 +34,10 @@
   <xacro:property name="left_prefix" value="${left_arm_prefix + '_' if left_arm_prefix else ''}"/>
   <xacro:property name="right_prefix" value="${right_arm_prefix + '_' if right_arm_prefix else ''}"/>
+  <link name="pnp_root"/>
+  <joint name="pnp_root_to_base_link" type="fixed">
+    <parent link="pnp_root"/>
+    <child link="base_link"/>
+    <origin xyz="0 0 0" rpy="0 0 0"/>
+  </joint>
   <link name="base_link">
     <visual>

Commit message: feat: update 45 degree mount base as default

File: pnp_dual_fr3_description/robots/pnp_dual_fr3/pnp_dual_fr3.srdf.xacro (robot description, xacro)
@@ -6,11 +6,15 @@
   <xacro:arg name="arm_prefixes" default="['left','right']"/>
   <xacro:property name="arm_prefixes_list" value="${$(arg arm_prefixes)}"/>
+  <xacro:arg name="mounting_type" default="dual_arm_45"/>
+  <xacro:arg name="home_pose_type" default="dual_arm_45"/>
   <xacro:arg name="hand" default="false"/>
   <xacro:arg name="ee_id" default="franka_hand"/>
   <xacro:property name="home_positions" value="${xacro.load_yaml('$(find pnp_dual_fr3_description)/config/home_positions.yaml')}"/>
+  <xacro:property name="selected_home_positions" value="${home_positions['$(arg home_pose_type)']}"/>
   <xacro:property name="left_prefix" value="${arm_prefixes_list[0] + '_' if arm_prefixes_list[0] else ''}"/>
   <xacro:property name="right_prefix" value="${arm_prefixes_list[1] + '_' if arm_prefixes_list[1] else ''}"/>
   <xacro:property name="left_full_prefix" value="${left_prefix + robot_types_list[0] + '_'}"/>
   <xacro:property name="right_full_prefix" value="${right_prefix + robot_types_list[1] + '_'}"/>
+  <xacro:property name="mounting_base_link" value="${'dual_arm_45_base_link' if '$(arg mounting_type)' == 'dual_arm_45' else 'base_link'}"/>
   <xacro:macro name="standard_arm_collisions" params="full_arm_prefix">
     <disable_collisions link1="${full_arm_prefix}link0" link2="${full_arm_prefix}link1" reason="Adjacent"/>
@@ -93,36 +97,36 @@
   </group_state>
   <group_state name="home" group="left_arm">
-    <joint name="${left_full_prefix}joint1" value="${home_positions.left.joint1}"/>
-    <joint name="${left_full_prefix}joint2" value="${home_positions.left.joint2}"/>
-    <joint name="${left_full_prefix}joint3" value="${home_positions.left.joint3}"/>
-    <joint name="${left_full_prefix}joint4" value="${home_positions.left.joint4}"/>
-    <joint name="${left_full_prefix}joint5" value="${home_positions.left.joint5}"/>
-    <joint name="${left_full_prefix}joint6" value="${home_positions.left.joint6}"/>
-    <joint name="${left_full_prefix}joint7" value="${home_positions.left.joint7}"/>
+    <joint name="${left_full_prefix}joint1" value="${selected_home_positions.left.joint1}"/>
+    <joint name="${left_full_prefix}joint2" value="${selected_home_positions.left.joint2}"/>
+    <joint name="${left_full_prefix}joint3" value="${selected_home_positions.left.joint3}"/>
+    <joint name="${left_full_prefix}joint4" value="${selected_home_positions.left.joint4}"/>
+    <joint name="${left_full_prefix}joint5" value="${selected_home_positions.left.joint5}"/>
+    <joint name="${left_full_prefix}joint6" value="${selected_home_positions.left.joint6}"/>
+    <joint name="${left_full_prefix}joint7" value="${selected_home_positions.left.joint7}"/>
   </group_state>
   <group_state name="home" group="right_arm">
-    <joint name="${right_full_prefix}joint1" value="${home_positions.right.joint1}"/>
-    <joint name="${right_full_prefix}joint2" value="${home_positions.right.joint2}"/>
-    <joint name="${right_full_prefix}joint3" value="${home_positions.right.joint3}"/>
-    <joint name="${right_full_prefix}joint4" value="${home_positions.right.joint4}"/>
-    <joint name="${right_full_prefix}joint5" value="${home_positions.right.joint5}"/>
-    <joint name="${right_full_prefix}joint6" value="${home_positions.right.joint6}"/>
-    <joint name="${right_full_prefix}joint7" value="${home_positions.right.joint7}"/>
+    <joint name="${right_full_prefix}joint1" value="${selected_home_positions.right.joint1}"/>
+    <joint name="${right_full_prefix}joint2" value="${selected_home_positions.right.joint2}"/>
+    <joint name="${right_full_prefix}joint3" value="${selected_home_positions.right.joint3}"/>
+    <joint name="${right_full_prefix}joint4" value="${selected_home_positions.right.joint4}"/>
+    <joint name="${right_full_prefix}joint5" value="${selected_home_positions.right.joint5}"/>
+    <joint name="${right_full_prefix}joint6" value="${selected_home_positions.right.joint6}"/>
+    <joint name="${right_full_prefix}joint7" value="${selected_home_positions.right.joint7}"/>
   </group_state>
   <group_state name="home" group="both_arms">
-    <joint name="${left_full_prefix}joint1" value="${home_positions.left.joint1}"/>
-    <joint name="${left_full_prefix}joint2" value="${home_positions.left.joint2}"/>
-    <joint name="${left_full_prefix}joint3" value="${home_positions.left.joint3}"/>
-    <joint name="${left_full_prefix}joint4" value="${home_positions.left.joint4}"/>
-    <joint name="${left_full_prefix}joint5" value="${home_positions.left.joint5}"/>
-    <joint name="${left_full_prefix}joint6" value="${home_positions.left.joint6}"/>
-    <joint name="${left_full_prefix}joint7" value="${home_positions.left.joint7}"/>
-    <joint name="${right_full_prefix}joint1" value="${home_positions.right.joint1}"/>
-    <joint name="${right_full_prefix}joint2" value="${home_positions.right.joint2}"/>
-    <joint name="${right_full_prefix}joint3" value="${home_positions.right.joint3}"/>
-    <joint name="${right_full_prefix}joint4" value="${home_positions.right.joint4}"/>
-    <joint name="${right_full_prefix}joint5" value="${home_positions.right.joint5}"/>
-    <joint name="${right_full_prefix}joint6" value="${home_positions.right.joint6}"/>
-    <joint name="${right_full_prefix}joint7" value="${home_positions.right.joint7}"/>
+    <joint name="${left_full_prefix}joint1" value="${selected_home_positions.left.joint1}"/>
+    <joint name="${left_full_prefix}joint2" value="${selected_home_positions.left.joint2}"/>
+    <joint name="${left_full_prefix}joint3" value="${selected_home_positions.left.joint3}"/>
+    <joint name="${left_full_prefix}joint4" value="${selected_home_positions.left.joint4}"/>
+    <joint name="${left_full_prefix}joint5" value="${selected_home_positions.left.joint5}"/>
+    <joint name="${left_full_prefix}joint6" value="${selected_home_positions.left.joint6}"/>
+    <joint name="${left_full_prefix}joint7" value="${selected_home_positions.left.joint7}"/>
+    <joint name="${right_full_prefix}joint1" value="${selected_home_positions.right.joint1}"/>
+    <joint name="${right_full_prefix}joint2" value="${selected_home_positions.right.joint2}"/>
+    <joint name="${right_full_prefix}joint3" value="${selected_home_positions.right.joint3}"/>
+    <joint name="${right_full_prefix}joint4" value="${selected_home_positions.right.joint4}"/>
+    <joint name="${right_full_prefix}joint5" value="${selected_home_positions.right.joint5}"/>
+    <joint name="${right_full_prefix}joint6" value="${selected_home_positions.right.joint6}"/>
+    <joint name="${right_full_prefix}joint7" value="${selected_home_positions.right.joint7}"/>
   </group_state>
   <virtual_joint name="world_joint" type="fixed" parent_frame="world" child_link="pnp_root"/>
@@ -131,14 +135,14 @@
   <xacro:standard_arm_collisions full_arm_prefix="${right_full_prefix}"/>
   <xacro:extra_arm_collisions full_arm_prefix="${right_full_prefix}"/>
-  <disable_collisions link1="base_link" link2="${left_full_prefix}link0" reason="Adjacent"/>
-  <disable_collisions link1="base_link" link2="${left_full_prefix}link1" reason="Never"/>
-  <disable_collisions link1="base_link" link2="${left_full_prefix}link2" reason="Never"/>
-  <disable_collisions link1="base_link" link2="${left_full_prefix}link3" reason="Never"/>
-  <disable_collisions link1="base_link" link2="${left_full_prefix}link4" reason="Never"/>
-  <disable_collisions link1="base_link" link2="${right_full_prefix}link0" reason="Adjacent"/>
-  <disable_collisions link1="base_link" link2="${right_full_prefix}link1" reason="Never"/>
-  <disable_collisions link1="base_link" link2="${right_full_prefix}link2" reason="Never"/>
-  <disable_collisions link1="base_link" link2="${right_full_prefix}link3" reason="Never"/>
-  <disable_collisions link1="base_link" link2="${right_full_prefix}link4" reason="Never"/>
+  <disable_collisions link1="${mounting_base_link}" link2="${left_full_prefix}link0" reason="Adjacent"/>
+  <disable_collisions link1="${mounting_base_link}" link2="${left_full_prefix}link1" reason="Never"/>
+  <disable_collisions link1="${mounting_base_link}" link2="${left_full_prefix}link2" reason="Never"/>
+  <disable_collisions link1="${mounting_base_link}" link2="${left_full_prefix}link3" reason="Never"/>
+  <disable_collisions link1="${mounting_base_link}" link2="${left_full_prefix}link4" reason="Never"/>
+  <disable_collisions link1="${mounting_base_link}" link2="${right_full_prefix}link0" reason="Adjacent"/>
+  <disable_collisions link1="${mounting_base_link}" link2="${right_full_prefix}link1" reason="Never"/>
+  <disable_collisions link1="${mounting_base_link}" link2="${right_full_prefix}link2" reason="Never"/>
+  <disable_collisions link1="${mounting_base_link}" link2="${right_full_prefix}link3" reason="Never"/>
+  <disable_collisions link1="${mounting_base_link}" link2="${right_full_prefix}link4" reason="Never"/>
   <xacro:cross_arm_loop left_idx="0" right_idx_start="0" right_idx_end="4"/>
   <xacro:cross_arm_loop left_idx="1" right_idx_start="0" right_idx_end="4"/>

File: pnp_dual_fr3_description/robots/pnp_dual_fr3/pnp_dual_fr3.urdf.xacro (robot description, xacro)
@@ -9,4 +9,6 @@
   <xacro:arg name="robot_ips" default="['172.16.0.2','172.16.0.3']"/>
   <xacro:property name="robot_ips_list" value="${$(arg robot_ips)}"/>
+  <xacro:arg name="mounting_type" default="dual_arm_45"/>
+  <xacro:arg name="home_pose_type" default="dual_arm_45"/>
   <xacro:arg name="no_prefix" default="false"/>
   <xacro:arg name="hand" default="false"/>
@@ -36,4 +38,5 @@
   <xacro:arg name="collision_behavior_upper_force_thresholds_nominal" default=""/>
   <xacro:property name="home_positions" value="${xacro.load_yaml('$(find pnp_dual_fr3_description)/config/home_positions.yaml')}"/>
+  <xacro:property name="selected_home_positions" value="${home_positions['$(arg home_pose_type)']}"/>
   <xacro:property name="left_robot_type" value="${robot_types_list[0]}"/>
   <xacro:property name="right_robot_type" value="${robot_types_list[1]}"/>
@@ -42,36 +45,54 @@
   <xacro:property name="left_prefix" value="${left_arm_prefix + '_' if left_arm_prefix else ''}"/>
   <xacro:property name="right_prefix" value="${right_arm_prefix + '_' if right_arm_prefix else ''}"/>
+  <xacro:property name="use_dual_arm_45_mounting" value="${'$(arg mounting_type)' == 'dual_arm_45'}"/>
+  <xacro:property name="mounting_base_link" value="${'dual_arm_45_base_link' if use_dual_arm_45_mounting else 'base_link'}"/>
+  <xacro:property name="mounting_base_mesh" value="${'dual_arm_45_base_link.STL' if use_dual_arm_45_mounting else 'base_link.STL'}"/>
+  <xacro:property name="mounting_base_visual_rpy" value="${'-1.5708000001 -0.0000000001 -3.1415853072' if use_dual_arm_45_mounting else '0 0 0'}"/>
+  <xacro:property name="left_mount_xyz" value="${'-0.038 0.18 0.304' if use_dual_arm_45_mounting else '-0.038 0.118 0.65'}"/>
+  <xacro:property name="left_mount_rpy" value="${'0.5567600306 0.5689773370 2.4626595739' if use_dual_arm_45_mounting else '1.57079265 2.35619449 3.14159265'}"/>
+  <xacro:property name="right_mount_xyz" value="${'-0.038 -0.18 0.304' if use_dual_arm_45_mounting else '-0.038 -0.118 0.65'}"/>
+  <xacro:property name="right_mount_rpy" value="${'-0.5567600306 0.5689773370 -2.4626595739' if use_dual_arm_45_mounting else '-1.57079265 2.35619449 -3.14159265'}"/>
   <link name="pnp_root"/>
-  <joint name="pnp_root_to_base_link" type="fixed">
+  <joint name="pnp_root_to_${mounting_base_link}" type="fixed">
     <parent link="pnp_root"/>
-    <child link="base_link"/>
+    <child link="${mounting_base_link}"/>
     <origin xyz="0 0 0" rpy="0 0 0"/>
   </joint>
-  <link name="base_link">
+  <link name="${mounting_base_link}">
     <visual>
+      <origin xyz="0 0 0" rpy="${mounting_base_visual_rpy}"/>
       <geometry>
-        <mesh filename="package://pnp_dual_fr3_description/meshes/base_link.STL"/>
+        <mesh filename="package://pnp_dual_fr3_description/meshes/${mounting_base_mesh}"/>
       </geometry>
     </visual>
     <collision>
+      <origin xyz="0 0 0" rpy="${mounting_base_visual_rpy}"/>
       <geometry>
-        <mesh filename="package://pnp_dual_fr3_description/meshes/base_link.STL"/>
+        <mesh filename="package://pnp_dual_fr3_description/meshes/${mounting_base_mesh}"/>
       </geometry>
     </collision>
-    <inertial>
-      <origin xyz="0.16881 6.9204e-06 -0.041149" rpy="0 0 0"/>
-      <mass value="126.89"/>
-      <inertia ixx="13.035" ixy="2.2312e-05" ixz="0.0074177" iyy="9.5179" iyz="-0.00013636" izz="16.483"/>
-    </inertial>
+    <xacro:if value="${use_dual_arm_45_mounting}">
+      <inertial>
+        <origin xyz="-0.0198650146477697 1.2755017047279E-05 0.222334575056727" rpy="0 0 0"/>
+        <mass value="6.60648599522062"/>
+        <inertia ixx="0.0936597875943432" ixy="1.09875644923452E-05" ixz="0.000154650545694182" iyy="0.0511056842352335" iyz="-1.54662487107246E-05" izz="0.0741382717847405"/>
+      </inertial>
+    </xacro:if>
+    <xacro:unless value="${use_dual_arm_45_mounting}">
+      <inertial>
+        <origin xyz="0.16881 6.9204e-06 -0.041149" rpy="0 0 0"/>
+        <mass value="126.89"/>
+        <inertia ixx="13.035" ixy="2.2312e-05" ixz="0.0074177" iyy="9.5179" iyz="-0.00013636" izz="16.483"/>
+      </inertial>
+    </xacro:unless>
   </link>
-  <!-- Mount transforms copied from dual_franka_linker_from_mjcf_curobo_fixed.urdf. -->
-  <joint name="base_link_to_${left_arm_prefix}_base" type="fixed">
-    <origin xyz="-0.038 0.118 0.65" rpy="1.57079265 2.35619449 3.14159265"/>
-    <parent link="base_link"/>
+  <joint name="${mounting_base_link}_to_${left_arm_prefix}_base" type="fixed">
+    <origin xyz="${left_mount_xyz}" rpy="${left_mount_rpy}"/>
+    <parent link="${mounting_base_link}"/>
     <child link="${left_arm_prefix}_base"/>
   </joint>
-  <joint name="base_link_to_${right_arm_prefix}_base" type="fixed">
-    <origin xyz="-0.038 -0.118 0.65" rpy="-1.57079265 2.35619449 -3.14159265"/>
-    <parent link="base_link"/>
+  <joint name="${mounting_base_link}_to_${right_arm_prefix}_base" type="fixed">
+    <origin xyz="${right_mount_xyz}" rpy="${right_mount_rpy}"/>
+    <parent link="${mounting_base_link}"/>
     <child link="${right_arm_prefix}_base"/>
   </joint>
@@ -126,5 +147,5 @@
       robot_type="${left_robot_type}"
       robot_ip="${robot_ips_list[0]}"
-      initial_positions="${home_positions.left}"
+      initial_positions="${selected_home_positions.left}"
       use_fake_hardware="$(arg use_fake_hardware)"
       fake_sensor_commands="$(arg fake_sensor_commands)"
@@ -146,5 +167,5 @@
       robot_type="${right_robot_type}"
       robot_ip="${robot_ips_list[1]}"
-      initial_positions="${home_positions.right}"
+      initial_positions="${selected_home_positions.right}"
       use_fake_hardware="$(arg use_fake_hardware)"
       fake_sensor_commands="$(arg fake_sensor_commands)"
