Commit message: feat: add home pose when using fake hardware

File: pnp_dual_fr3_description/robots/pnp_dual_fr3/pnp_dual_fr3.urdf.xacro (robot description, xacro)
@@ -2,4 +2,5 @@
 <robot xmlns:xacro="http://www.ros.org/wiki/xacro" name="pnp_dual_fr3">
   <xacro:include filename="$(find franka_description)/robots/common/franka_robot.xacro"/>
+  <xacro:include filename="$(find pnp_dual_fr3_description)/robots/pnp_dual_fr3/pnp_dual_fr3.ros2_control.xacro"/>
   <xacro:arg name="robot_types" default="['fr3v2','fr3v2']"/>
   <xacro:property name="robot_types_list" value="${$(arg robot_types)}"/>
@@ -26,4 +27,5 @@
   <xacro:arg name="is_async" default="false"/>
   <xacro:arg name="thread_priority" default="50"/>
+  <xacro:property name="home_positions" value="${xacro.load_yaml('$(find pnp_dual_fr3_description)/config/home_positions.yaml')}"/>
   <xacro:property name="left_robot_type" value="${robot_types_list[0]}"/>
   <xacro:property name="right_robot_type" value="${robot_types_list[1]}"/>
@@ -38,17 +40,7 @@
       </geometry>
     </visual>
-    <visual>
-      <geometry>
-        <mesh filename="package://pnp_dual_fr3_description/meshes/adapter.stl" scale="0.001 0.001 0.001"/>
-      </geometry>
-    </visual>
     <collision>
       <geometry>
         <mesh filename="package://pnp_dual_fr3_description/meshes/base_link.STL"/>
-      </geometry>
-    </collision>
-    <collision>
-      <geometry>
-        <mesh filename="package://pnp_dual_fr3_description/meshes/adapter.stl" scale="0.001 0.001 0.001"/>
       </geometry>
     </collision>
@@ -87,5 +79,5 @@
     safety_distance="$(arg safety_distance)"
     with_sc="$(arg with_sc)"
-    ros2_control="$(arg ros2_control)"
+    ros2_control="false"
     robot_ip="${robot_ips_list[0]}"
     use_fake_hardware="$(arg use_fake_hardware)"
@@ -115,5 +107,5 @@
     safety_distance="$(arg safety_distance)"
     with_sc="$(arg with_sc)"
-    ros2_control="$(arg ros2_control)"
+    ros2_control="false"
     robot_ip="${robot_ips_list[1]}"
     use_fake_hardware="$(arg use_fake_hardware)"
@@ -126,3 +118,29 @@
     is_async="$(arg is_async)"
     thread_priority="$(arg thread_priority)"/>
+  <xacro:if value="$(arg ros2_control)">
+    <xacro:pnp_franka_arm_ros2_control
+      robot_type="${left_robot_type}"
+      robot_ip="${robot_ips_list[0]}"
+      initial_positions="${home_positions.left}"
+      use_fake_hardware="$(arg use_fake_hardware)"
+      fake_sensor_commands="$(arg fake_sensor_commands)"
+      gazebo="$(arg gazebo)"
+      hand="$(arg hand)"
+      gazebo_effort="$(arg gazebo_effort)"
+      arm_prefix="${left_prefix}"
+      is_async="$(arg is_async)"
+      thread_priority="$(arg thread_priority)"/>
+    <xacro:pnp_franka_arm_ros2_control
+      robot_type="${right_robot_type}"
+      robot_ip="${robot_ips_list[1]}"
+      initial_positions="${home_positions.right}"
+      use_fake_hardware="$(arg use_fake_hardware)"
+      fake_sensor_commands="$(arg fake_sensor_commands)"
+      gazebo="$(arg gazebo)"
+      hand="$(arg hand)"
+      gazebo_effort="$(arg gazebo_effort)"
+      arm_prefix="${right_prefix}"
+      is_async="$(arg is_async)"
+      thread_priority="$(arg thread_priority)"/>
+  </xacro:if>
 </robot>

File: pnp_dual_fr3_moveit_config/config/pnp_dual_fr3.srdf.xacro (robot description, xacro)
@@ -8,4 +8,5 @@
   <xacro:arg name="hand" default="false"/>
   <xacro:arg name="ee_id" default="franka_hand"/>
+  <xacro:property name="home_positions" value="${xacro.load_yaml('$(find pnp_dual_fr3_description)/config/home_positions.yaml')}"/>
   <xacro:property name="left_prefix" value="${arm_prefixes_list[0] + '_' if arm_prefixes_list[0] else ''}"/>
   <xacro:property name="right_prefix" value="${arm_prefixes_list[1] + '_' if arm_prefixes_list[1] else ''}"/>
@@ -91,4 +92,38 @@
     <joint name="${right_full_prefix}joint7" value="${pi/4}"/>
   </group_state>
+  <group_state name="home" group="left_arm">
+    <joint name="${left_full_prefix}joint1" value="${home_positions.left.joint1}"/>
+    <joint name="${left_full_prefix}joint2" value="${home_positions.left.joint2}"/>
+    <joint name="${left_full_prefix}joint3" value="${home_positions.left.joint3}"/>
+    <joint name="${left_full_prefix}joint4" value="${home_positions.left.joint4}"/>
+    <joint name="${left_full_prefix}joint5" value="${home_positions.left.joint5}"/>
+    <joint name="${left_full_prefix}joint6" value="${home_positions.left.joint6}"/>
+    <joint name="${left_full_prefix}joint7" value="${home_positions.left.joint7}"/>
+  </group_state>
+  <group_state name="home" group="right_arm">
+    <joint name="${right_full_prefix}joint1" value="${home_positions.right.joint1}"/>
+    <joint name="${right_full_prefix}joint2" value="${home_positions.right.joint2}"/>
+    <joint name="${right_full_prefix}joint3" value="${home_positions.right.joint3}"/>
+    <joint name="${right_full_prefix}joint4" value="${home_positions.right.joint4}"/>
+    <joint name="${right_full_prefix}joint5" value="${home_positions.right.joint5}"/>
+    <joint name="${right_full_prefix}joint6" value="${home_positions.right.joint6}"/>
+    <joint name="${right_full_prefix}joint7" value="${home_positions.right.joint7}"/>
+  </group_state>
+  <group_state name="home" group="both_arms">
+    <joint name="${left_full_prefix}joint1" value="${home_positions.left.joint1}"/>
+    <joint name="${left_full_prefix}joint2" value="${home_positions.left.joint2}"/>
+    <joint name="${left_full_prefix}joint3" value="${home_positions.left.joint3}"/>
+    <joint name="${left_full_prefix}joint4" value="${home_positions.left.joint4}"/>
+    <joint name="${left_full_prefix}joint5" value="${home_positions.left.joint5}"/>
+    <joint name="${left_full_prefix}joint6" value="${home_positions.left.joint6}"/>
+    <joint name="${left_full_prefix}joint7" value="${home_positions.left.joint7}"/>
+    <joint name="${right_full_prefix}joint1" value="${home_positions.right.joint1}"/>
+    <joint name="${right_full_prefix}joint2" value="${home_positions.right.joint2}"/>
+    <joint name="${right_full_prefix}joint3" value="${home_positions.right.joint3}"/>
+    <joint name="${right_full_prefix}joint4" value="${home_positions.right.joint4}"/>
+    <joint name="${right_full_prefix}joint5" value="${home_positions.right.joint5}"/>
+    <joint name="${right_full_prefix}joint6" value="${home_positions.right.joint6}"/>
+    <joint name="${right_full_prefix}joint7" value="${home_positions.right.joint7}"/>
+  </group_state>
   <virtual_joint name="world_joint" type="fixed" parent_frame="world" child_link="base_link"/>
   <xacro:standard_arm_collisions full_arm_prefix="${left_full_prefix}"/>

Commit message: feat: fix urdf mount

File: pnp_dual_fr3_description/robots/pnp_dual_fr3/pnp_dual_fr3.urdf.xacro (robot description, xacro)
@@ -53,10 +53,10 @@
   <!-- Mount transforms copied from dual_franka_linker_from_mjcf_curobo_fixed.urdf. -->
   <joint name="base_link_to_${left_arm_prefix}_base" type="fixed">
-    <origin xyz="-0.038 0.118 0.65" rpy="1.57079265 0.786592654 3.14159265"/>
+    <origin xyz="-0.038 0.118 0.65" rpy="1.57079265 2.35619449 3.14159265"/>
     <parent link="base_link"/>
     <child link="${left_arm_prefix}_base"/>
   </joint>
   <joint name="base_link_to_${right_arm_prefix}_base" type="fixed">
-    <origin xyz="-0.038 -0.118 0.65" rpy="-1.57079265 0.786592654 -3.14159265"/>
+    <origin xyz="-0.038 -0.118 0.65" rpy="-1.57079265 2.35619449 -3.14159265"/>
     <parent link="base_link"/>
     <child link="${right_arm_prefix}_base"/>

Commit message: feat: update pnp 45 degree urdf

File: pnp_dual_fr3_description/robots/pnp_dual_fr3/pnp_dual_fr3.urdf.xacro (robot description, xacro)
@@ -48,14 +48,15 @@
   <xacro:property name="mounting_base_link" value="${'dual_arm_45_base_link' if use_dual_arm_45_mounting else 'base_link'}"/>
   <xacro:property name="mounting_base_mesh" value="${'dual_arm_45_base_link.STL' if use_dual_arm_45_mounting else 'base_link.STL'}"/>
+  <xacro:property name="mounting_base_origin_rpy" value="${'0 0 0' if use_dual_arm_45_mounting else '0 0 0'}"/>
   <xacro:property name="mounting_base_visual_rpy" value="${'-1.5708000001 -0.0000000001 -3.1415853072' if use_dual_arm_45_mounting else '0 0 0'}"/>
-  <xacro:property name="left_mount_xyz" value="${'-0.038 0.18 0.304' if use_dual_arm_45_mounting else '-0.038 0.118 0.65'}"/>
-  <xacro:property name="left_mount_rpy" value="${'0.5567600306 0.5689773370 2.4626595739' if use_dual_arm_45_mounting else '1.57079265 2.35619449 3.14159265'}"/>
-  <xacro:property name="right_mount_xyz" value="${'-0.038 -0.18 0.304' if use_dual_arm_45_mounting else '-0.038 -0.118 0.65'}"/>
-  <xacro:property name="right_mount_rpy" value="${'-0.5567600306 0.5689773370 -2.4626595739' if use_dual_arm_45_mounting else '-1.57079265 2.35619449 -3.14159265'}"/>
+  <xacro:property name="left_mount_xyz" value="${'-0.038 -0.18 0.304' if use_dual_arm_45_mounting else '-0.038 0.118 0.65'}"/>
+  <xacro:property name="left_mount_rpy" value="${'-0.5567600306 0.5689773370 -2.4626595739' if use_dual_arm_45_mounting else '1.57079265 2.35619449 3.14159265'}"/>
+  <xacro:property name="right_mount_xyz" value="${'-0.038 0.18 0.304' if use_dual_arm_45_mounting else '-0.038 -0.118 0.65'}"/>
+  <xacro:property name="right_mount_rpy" value="${'0.5567600306 0.5689773370 2.4626595739' if use_dual_arm_45_mounting else '-1.57079265 2.35619449 -3.14159265'}"/>
   <link name="pnp_root"/>
   <joint name="pnp_root_to_${mounting_base_link}" type="fixed">
     <parent link="pnp_root"/>
     <child link="${mounting_base_link}"/>
-    <origin xyz="0 0 0" rpy="0 0 0"/>
+    <origin xyz="0 0 0" rpy="${mounting_base_origin_rpy}"/>
   </joint>
   <link name="${mounting_base_link}">
